Commit message: divisione nodo superpoint

File: urdf/robopy.urdf (robot description, URDF)
Before this commit: robot tracked_robot, 6 links, 5 joints
Links:
- removed link camera_frame
- removed link camera_link
- added link imu_link
- added link oak_mount_link
- link base_link: mass 5 -> 5.0; geometry collision box size=0.20 0.20 0.15; visual box size=0.20 0.20 0.15
- link left_track: mass 1 -> None; geometry 
- link right_track: mass 1 -> None; geometry 
- link ultrasonic_link: geometry 
Joints:
- removed joint camera_frame_joint
- removed joint camera_joint
- added joint imu_joint: type fixed, parent base_link, child imu_link, origin xyz=0.10 0.0 0.15 rpy=0 0 0
- added joint oak_mount_joint: type fixed, parent base_link, child oak_mount_link, origin xyz=0.10 0.0 0.15 rpy=0 -0.1535 0
- joint left_track_joint: axis 0 1 0 -> (none); origin xyz=0 0.1 0 rpy=0 1.5708 0 -> xyz=0 0.08 0.05 rpy=0 0 0; type continuous -> fixed
- joint right_track_joint: axis 0 1 0 -> (none); origin xyz=0 -0.1 0 rpy=0 1.5708 0 -> xyz=0 -0.08 0.05 rpy=0 0 0; type continuous -> fixed
- joint ultrasonic_joint: origin xyz=0.1 0.0 0.02 rpy=1.5708 0 0 -> xyz=0.10 0.0 0.05 rpy=1.5708 0 0

Commit message: feat: Integrate RTAB-Map, configure Nav2 with MPPI controller, add visual exploration skill, and introduce smart buildhat driver with related system updates.

File: urdf/robopy.urdf (robot description, URDF)
Before this commit: robot tracked_robot, 6 links, 5 joints
Links:
- link base_link: geometry collision box size=0.20 0.20 0.15; visual mesh filename=package://robopy_controller/urdf/Marcus.stl scale=0.001 0.001 0.001

Commit message: docs: implement Book-to-Skill documentation refactoring and update system configuration and nodes

File: urdf/robopy.urdf (robot description, URDF)
Before this commit: robot tracked_robot, 6 links, 5 joints
Links:
- removed link oak_mount_link
- added link camera_link
- added link camera_optical_frame
Joints:
- removed joint oak_mount_joint
- added joint camera_joint: type fixed, parent base_link, child camera_link, origin xyz=0.05 0.0 0.08 rpy=0 -0.1535 0
- added joint camera_optical_joint: type fixed, parent camera_link, child camera_optical_frame, origin xyz=0 0 0 rpy=-1.5708 0 -1.5708
