Commit message: fix(tf): set camera pitch to -0.1396 rad (-8 deg UP) in restart_hailo.sh and URDF

File: urdf/robopy.urdf (robot description, URDF)
Before this commit: robot tracked_robot, 7 links, 6 joints
Joints:
- joint camera_joint: origin xyz=0.05 0.0 0.08 rpy=0 -0.1535 0 -> xyz=0.0332 0.0 0.2616 rpy=0 -0.1396 0

Commit message: fix(vui): resolve conversational gating, restore non-destructive <IGNORE_TURN> and 110.0 RMS pre-gate (FM-VUI-044, ECO-2026-10-11-001)

File: urdf/robopy.urdf (robot description, URDF)
Before this commit: robot tracked_robot, 7 links, 6 joints
Links:
- removed link camera_link
- removed link ultrasonic_link
- added link base_footprint
- added link chassis_imu_link
- added link laser; visual cylinder length=0.04 radius=0.032
- added link oak_camera_link; visual box size=0.02 0.09 0.03
- added link oak_imu_frame
- added link oak_left_camera_optical_frame
- added link ultrasonic_sensor
- link base_link: mass 5.0 -> None; geometry collision box size=0.25 0.22 0.12; visual box size=0.25 0.22 0.12
- link left_track: geometry visual cylinder length=0.04 radius=0.0335
- link right_track: geometry visual cylinder length=0.04 radius=0.0335
Joints:
- removed joint camera_joint
- removed joint ultrasonic_joint
- added joint base_footprint_joint: type fixed, parent base_link, child base_footprint, origin xyz=0 0 -0.0335 rpy=0 0 0
- added joint chassis_imu_joint: type fixed, parent base_link, child chassis_imu_link, origin xyz=0.0 0.0 0.05 rpy=0 0 0
- added joint laser_joint: type fixed, parent base_link, child laser, origin xyz=0.08 0.0 0.18 rpy=0.0 0.0 3.14159265
- added joint oak_camera_joint: type fixed, parent base_link, child oak_camera_link, origin xyz=0.0332 0.0 0.2616 rpy=0.0 -0.1396 0.0
- added joint oak_imu_joint: type fixed, parent oak_camera_link, child oak_imu_frame, origin xyz=0 0 0 rpy=0 0 0
- added joint oak_left_camera_optical_joint: type fixed, parent oak_camera_link, child oak_left_camera_optical_frame, origin xyz=0 0 0 rpy=-1.5708 0.0 -1.5708
- added joint ultrasonic_sensor_joint: type fixed, parent base_link, child ultrasonic_sensor, origin xyz=0.12 0.0 0.05 rpy=0 0 0
- joint camera_optical_joint: origin xyz=0 0 0 rpy=-1.5708 0 -1.5708 -> xyz=0 0 0 rpy=-1.5708 0.0 -1.5708; parent camera_link -> oak_camera_link
- joint left_track_joint: origin xyz=0 0.08 0.05 rpy=0 0 0 -> xyz=0 0.1425 0.0 rpy=0 0 0
- joint right_track_joint: origin xyz=0 -0.08 0.05 rpy=0 0 0 -> xyz=0 -0.1425 0.0 rpy=0 0 0
